File: output/pcbs/travis_erg2026.kicad_pcb (KiCad board)
At the start: 2 copper layers, 161.3 x 139.9 mm, 85 parts

Commit message: leds
Parts:
- added C1: 10V 1000uF, Capacitor_THT:C_Radial_D6.3mm_H11.0mm_P2.50mm, B.Cu at (163.3, 80.1)
- added C10: C_1206_3216Metric, C_1206_3216Metric, B.Cu at (82.8, 109.4)
- added C11: C_1206_3216Metric, C_1206_3216Metric, B.Cu at (104.4, 192.3)
- added C12: C_1206_3216Metric, C_1206_3216Metric, B.Cu at (104.4, 150.2)
- added C13: C_1206_3216Metric, C_1206_3216Metric, B.Cu at (104.4, 108.1)
- added C14: C_1206_3216Metric, C_1206_3216Metric, B.Cu at (124.4, 193.4)
- added C15: C_1206_3216Metric, C_1206_3216Metric, B.Cu at (125.2, 151.3)
- added C16: C_1206_3216Metric, C_1206_3216Metric, B.Cu at (125.9, 109.2)
- added C17: C_1206_3216Metric, C_1206_3216Metric, B.Cu at (144.5, 194.8)
- added C18: C_1206_3216Metric, C_1206_3216Metric, B.Cu at (146.0, 152.8)
- added C19: C_1206_3216Metric, C_1206_3216Metric, B.Cu at (147.5, 110.7)
- added C2: C_1206_3216Metric, C_1206_3216Metric, B.Cu at (44.2, 197.2)
- added C20: C_1206_3216Metric, C_1206_3216Metric, B.Cu at (164.6, 196.6)
- added C21: C_1206_3216Metric, C_1206_3216Metric, B.Cu at (166.8, 154.6)
- added C22: C_1206_3216Metric, C_1206_3216Metric, B.Cu at (169.0, 112.5)
- added C23: C_1206_3216Metric, C_1206_3216Metric, B.Cu at (34.2, 171.9)
- added C24: C_1206_3216Metric, C_1206_3216Metric, B.Cu at (32.0, 129.8)
- added C25: C_1206_3216Metric, C_1206_3216Metric, B.Cu at (29.8, 87.8)
- added C26: C_1206_3216Metric, C_1206_3216Metric, B.Cu at (54.6, 169.7)
- added C27: C_1206_3216Metric, C_1206_3216Metric, B.Cu at (53.2, 127.6)
- added C28: C_1206_3216Metric, C_1206_3216Metric, B.Cu at (51.7, 85.6)
- added C29: C_1206_3216Metric, C_1206_3216Metric, B.Cu at (75.1, 167.9)
- added C3: C_1206_3216Metric, C_1206_3216Metric, B.Cu at (42.0, 155.2)
- added C30: C_1206_3216Metric, C_1206_3216Metric, B.Cu at (74.4, 125.8)
- added C31: C_1206_3216Metric, C_1206_3216Metric, B.Cu at (73.7, 83.7)
- added C32: C_1206_3216Metric, C_1206_3216Metric, B.Cu at (95.7, 166.5)
- added C33: C_1206_3216Metric, C_1206_3216Metric, B.Cu at (95.7, 124.4)
- added C34: C_1206_3216Metric, C_1206_3216Metric, B.Cu at (95.7, 82.3)
- added C35: C_1206_3216Metric, C_1206_3216Metric, B.Cu at (116.2, 167.4)
- added C36: C_1206_3216Metric, C_1206_3216Metric, B.Cu at (116.9, 125.3)
- added C37: C_1206_3216Metric, C_1206_3216Metric, B.Cu at (117.7, 83.2)
- added C38: C_1206_3216Metric, C_1206_3216Metric, B.Cu at (136.7, 168.7)
- added C39: C_1206_3216Metric, C_1206_3216Metric, B.Cu at (138.2, 126.6)
- added C4: C_1206_3216Metric, C_1206_3216Metric, B.Cu at (39.8, 113.1)
- added C40: C_1206_3216Metric, C_1206_3216Metric, B.Cu at (139.7, 84.6)
- added C41: C_1206_3216Metric, C_1206_3216Metric, B.Cu at (157.2, 170.4)
- added C42: C_1206_3216Metric, C_1206_3216Metric, B.Cu at (159.4, 128.3)
- added C43: C_1206_3216Metric, C_1206_3216Metric, B.Cu at (161.6, 86.3)
- added C5: C_1206_3216Metric, C_1206_3216Metric, B.Cu at (64.2, 195.2)
- added C6: C_1206_3216Metric, C_1206_3216Metric, B.Cu at (62.8, 153.2)
- added C7: C_1206_3216Metric, C_1206_3216Metric, B.Cu at (61.3, 111.1)
- added C8: C_1206_3216Metric, C_1206_3216Metric, B.Cu at (84.3, 193.6)
- added C9: C_1206_3216Metric, C_1206_3216Metric, B.Cu at (83.5, 151.5)
- added LED1: SK6812mini-e, travis:led_SK6812mini-e (per-key, single-side), B.Cu at (39.7, 195.0)
- added LED10: SK6812mini-e, travis:led_SK6812mini-e (per-key, single-side), B.Cu at (100.0, 189.9)
- added LED11: SK6812mini-e, travis:led_SK6812mini-e (per-key, single-side), B.Cu at (100.0, 147.8)
- added LED12: SK6812mini-e, travis:led_SK6812mini-e (per-key, single-side), B.Cu at (100.0, 105.7)
- added LED13: SK6812mini-e, travis:led_SK6812mini-e (per-key, single-side), B.Cu at (120.1, 190.9)
- added LED14: SK6812mini-e, travis:led_SK6812mini-e (per-key, single-side), B.Cu at (120.9, 148.9)
- added LED15: SK6812mini-e, travis:led_SK6812mini-e (per-key, single-side), B.Cu at (121.6, 106.8)
- added LED16: SK6812mini-e, travis:led_SK6812mini-e (per-key, single-side), B.Cu at (140.3, 192.3)
- added LED17: SK6812mini-e, travis:led_SK6812mini-e (per-key, single-side), B.Cu at (141.7, 150.2)
- added LED18: SK6812mini-e, travis:led_SK6812mini-e (per-key, single-side), B.Cu at (143.2, 108.1)
- added LED19: SK6812mini-e, travis:led_SK6812mini-e (per-key, single-side), B.Cu at (160.3, 194.0)
- added LED2: SK6812mini-e, travis:led_SK6812mini-e (per-key, single-side), B.Cu at (37.5, 153.0)
- added LED20: SK6812mini-e, travis:led_SK6812mini-e (per-key, single-side), B.Cu at (162.5, 152.0)
- added LED21: SK6812mini-e, travis:led_SK6812mini-e (per-key, single-side), B.Cu at (164.8, 109.9)
- added LED22: SK6812mini-e, travis:led_SK6812mini-e (per-key, single-side), B.Cu at (38.6, 174.0)
- added LED23: SK6812mini-e, travis:led_SK6812mini-e (per-key, single-side), B.Cu at (36.4, 132.0)
- added LED24: SK6812mini-e, travis:led_SK6812mini-e (per-key, single-side), B.Cu at (34.2, 89.9)
- added LED25: SK6812mini-e, travis:led_SK6812mini-e (per-key, single-side), B.Cu at (59.1, 172.0)
- added LED26: SK6812mini-e, travis:led_SK6812mini-e (per-key, single-side), B.Cu at (57.6, 129.9)
- added LED27: SK6812mini-e, travis:led_SK6812mini-e (per-key, single-side), B.Cu at (56.1, 87.8)
- added LED28: SK6812mini-e, travis:led_SK6812mini-e (per-key, single-side), B.Cu at (79.5, 170.2)
- added LED29: SK6812mini-e, travis:led_SK6812mini-e (per-key, single-side), B.Cu at (78.8, 128.2)
- added LED3: SK6812mini-e, travis:led_SK6812mini-e (per-key, single-side), B.Cu at (35.3, 111.0)
- added LED30: SK6812mini-e, travis:led_SK6812mini-e (per-key, single-side), B.Cu at (78.0, 86.1)
- added LED31: SK6812mini-e, travis:led_SK6812mini-e (per-key, single-side), B.Cu at (100.0, 168.9)
- added LED32: SK6812mini-e, travis:led_SK6812mini-e (per-key, single-side), B.Cu at (100.0, 126.8)
- added LED33: SK6812mini-e, travis:led_SK6812mini-e (per-key, single-side), B.Cu at (100.0, 84.7)
- added LED34: SK6812mini-e, travis:led_SK6812mini-e (per-key, single-side), B.Cu at (120.5, 169.9)
- added LED35: SK6812mini-e, travis:led_SK6812mini-e (per-key, single-side), B.Cu at (121.2, 127.8)
- added LED36: SK6812mini-e, travis:led_SK6812mini-e (per-key, single-side), B.Cu at (122.0, 85.7)
- added LED37: SK6812mini-e, travis:led_SK6812mini-e (per-key, single-side), B.Cu at (141.0, 171.3)
- added LED38: SK6812mini-e, travis:led_SK6812mini-e (per-key, single-side), B.Cu at (142.5, 129.2)
- added LED39: SK6812mini-e, travis:led_SK6812mini-e (per-key, single-side), B.Cu at (143.9, 87.1)
- added LED4: SK6812mini-e, travis:led_SK6812mini-e (per-key, single-side), B.Cu at (59.8, 193.0)
- added LED40: SK6812mini-e, travis:led_SK6812mini-e (per-key, single-side), B.Cu at (161.4, 173.0)
- added LED41: SK6812mini-e, travis:led_SK6812mini-e (per-key, single-side), B.Cu at (163.6, 130.9)
- added LED42: SK6812mini-e, travis:led_SK6812mini-e (per-key, single-side), B.Cu at (165.9, 88.9)
- added LED5: SK6812mini-e, travis:led_SK6812mini-e (per-key, single-side), B.Cu at (58.3, 150.9)
- added LED6: SK6812mini-e, travis:led_SK6812mini-e (per-key, single-side), B.Cu at (56.9, 108.8)
- added LED7: SK6812mini-e, travis:led_SK6812mini-e (per-key, single-side), B.Cu at (79.9, 191.3)
- added LED8: SK6812mini-e, travis:led_SK6812mini-e (per-key, single-side), B.Cu at (79.2, 149.2)
- added LED9: SK6812mini-e, travis:led_SK6812mini-e (per-key, single-side), B.Cu at (78.4, 107.1)
- MCU1: value (none) -> Arduino Pro Micro; footprint ProMicro -> Arduino_Pro_Micro
- moved MCU1 62.8 mm to (162.5, 95.7), turned to -93 degrees
Connections:
- net P0 renamed encA
- net P1 renamed encC
- net P10 renamed LED_0
- net P20 renamed scl
- net P21 renamed sda
- MCU1 pad 1: RAW -> D3
- MCU1 pad 10: P14 -> row3
- MCU1 pad 11: P16 -> row4
- MCU1 pad 15: GND -> B3
- MCU1 pad 16: GND -> B1
- MCU1 pad 17: P2 -> col3
- MCU1 pad 18: P3 -> col2
- MCU1 pad 19: P4 -> col1
- MCU1 pad 2: GND -> D2
- MCU1 pad 20: P5 -> col0
- MCU1 pad 21: P6 -> VCC
- MCU1 pad 22: P7 -> RST
- MCU1 pad 23: P8 -> GND
- MCU1 pad 24: P9 -> RAW
- MCU1 pad 3: RST -> GND
- MCU1 pad 4: VCC -> GND
- MCU1 pad 7: P19 -> row0
- MCU1 pad 8: P18 -> row1
- MCU1 pad 9: P15 -> row2
- S1 pad 2: outer2_mod -> matrix_outer2_mod
- S10 pad 2: outer1_top -> matrix_outer1_top
- S11 pad 2: outer1_num -> matrix_outer1_num
- S12 pad 2: outer1_func -> matrix_outer1_func
- S13 pad 2: pinky_mod -> matrix_pinky_mod
- S14 pad 2: pinky_bottom -> matrix_pinky_bottom
- S15 pad 2: pinky_home -> matrix_pinky_home
- S16 pad 2: pinky_top -> matrix_pinky_top
- S17 pad 2: pinky_num -> matrix_pinky_num
- S18 pad 2: pinky_func -> matrix_pinky_func
- S19 pad 2: ring_mod -> matrix_ring_mod
- S2 pad 2: outer2_bottom -> matrix_outer2_bottom
- S20 pad 2: ring_bottom -> matrix_ring_bottom
- S21 pad 2: ring_home -> matrix_ring_home
- S22 pad 2: ring_top -> matrix_ring_top
- S23 pad 2: ring_num -> matrix_ring_num
- S24 pad 2: ring_func -> matrix_ring_func
- S25 pad 2: middle_mod -> matrix_middle_mod
- S26 pad 2: middle_bottom -> matrix_middle_bottom
- S27 pad 2: middle_home -> matrix_middle_home
- S28 pad 2: middle_top -> matrix_middle_top
- S29 pad 2: middle_num -> matrix_middle_num
- S3 pad 2: outer2_home -> matrix_outer2_home
- S30 pad 2: middle_func -> matrix_middle_func
- S31 pad 2: index_mod -> matrix_index_mod
- S32 pad 2: index_bottom -> matrix_index_bottom
- S33 pad 2: index_home -> matrix_index_home
- S34 pad 2: index_top -> matrix_index_top
- S35 pad 2: index_num -> matrix_index_num
- S36 pad 2: index_func -> matrix_index_func
- S37 pad 2: inner_mod -> matrix_inner_mod
- S38 pad 2: inner_bottom -> matrix_inner_bottom
- S39 pad 2: inner_home -> matrix_inner_home
- S4 pad 2: outer2_top -> matrix_outer2_top
- S40 pad 2: inner_top -> matrix_inner_top
- S41 pad 2: inner_num -> matrix_inner_num
- S42 pad 2: inner_func -> matrix_inner_func
- S5 pad 2: outer2_num -> matrix_outer2_num
- S6 pad 2: outer2_func -> matrix_outer2_func
- S7 pad 2: outer1_mod -> matrix_outer1_mod
- S8 pad 2: outer1_bottom -> matrix_outer1_bottom
- S9 pad 2: outer1_home -> matrix_outer1_home

Commit message: pcb generation
Parts:
- added LOGO1: , ceoloide:utility_ergogen_logo, F.Cu at (87.8, 70.0)
- added LOGO2: , travis:travis, F.Cu at (132.3, 69.6)
- added ROC1: , travis:travis, B.Cu at (43.4, 73.9)
- C1: moved to F.Cu
- moved MCU1 25.4 mm to (173.2, 72.6)
- moved C22 23.8 mm to (180.1, 91.5), turned to 177 degrees
- moved LED21 23.8 mm to (175.9, 88.9), turned to 177 degrees
- moved C25 23.8 mm to (40.9, 108.8), turned to 3 degrees
- moved LED24 23.8 mm to (45.3, 111.0), turned to 3 degrees
- moved C20 23.8 mm to (175.7, 175.6), turned to 177 degrees
- moved C21 23.8 mm to (177.9, 133.6), turned to 177 degrees
- moved LED19 23.8 mm to (171.4, 173.0), turned to 177 degrees
- moved LED20 23.8 mm to (173.6, 130.9), turned to 177 degrees
- moved C23 23.8 mm to (45.3, 192.9), turned to 3 degrees
- moved C24 23.8 mm to (43.1, 150.8), turned to 3 degrees
- moved LED22 23.8 mm to (49.7, 195.0), turned to 3 degrees
- moved LED23 23.8 mm to (47.5, 153.0), turned to 3 degrees
- moved C17 23.6 mm to (155.3, 173.8), turned to 178 degrees
- moved C18 23.6 mm to (156.7, 131.7), turned to 178 degrees
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Connections:
- net LED_0 renamed B5
- net matrix_index_bottom renamed matrix_col5_row1
- net matrix_index_func renamed matrix_col5_row5
- net matrix_index_home renamed matrix_col5_row2
- net matrix_index_mod renamed matrix_col5_row0
- net matrix_index_num renamed matrix_col5_row4
- net matrix_index_top renamed matrix_col5_row3
- net matrix_inner_bottom renamed matrix_col6_row1
- net matrix_inner_func renamed matrix_col6_row5
- net matrix_inner_home renamed matrix_col6_row2
- net matrix_inner_mod renamed matrix_col6_row0
- net matrix_inner_num renamed matrix_col6_row4
- net matrix_inner_top renamed matrix_col6_row3
- net matrix_middle_bottom renamed matrix_col4_row1
- net matrix_middle_func renamed matrix_col4_row5
- net matrix_middle_home renamed matrix_col4_row2
- net matrix_middle_mod renamed matrix_col4_row0
- net matrix_middle_num renamed matrix_col4_row4
- net matrix_middle_top renamed matrix_col4_row3
- net matrix_outer1_bottom renamed matrix_col1_row1
- net matrix_outer1_func renamed matrix_col1_row5
- net matrix_outer1_home renamed matrix_col1_row2
- net matrix_outer1_mod renamed matrix_col1_row0
- net matrix_outer1_num renamed matrix_col1_row4
- net matrix_outer1_top renamed matrix_col1_row3
- net matrix_outer2_bottom renamed matrix_col0_row1
- net matrix_outer2_func renamed matrix_col0_row5
- net matrix_outer2_home renamed matrix_col0_row2
- net matrix_outer2_mod renamed matrix_col0_row0
- net matrix_outer2_num renamed matrix_col0_row4
- net matrix_outer2_top renamed matrix_col0_row3
- net matrix_pinky_bottom renamed matrix_col2_row1
- net matrix_pinky_func renamed matrix_col2_row5
- net matrix_pinky_home renamed matrix_col2_row2
- net matrix_pinky_mod renamed matrix_col2_row0
- net matrix_pinky_num renamed matrix_col2_row4
- net matrix_pinky_top renamed matrix_col2_row3
- net matrix_ring_bottom renamed matrix_col3_row1
- net matrix_ring_func renamed matrix_col3_row5
- net matrix_ring_home renamed matrix_col3_row2
- net matrix_ring_mod renamed matrix_col3_row0
- net matrix_ring_num renamed matrix_col3_row4
- net matrix_ring_top renamed matrix_col3_row3
- net sda renamed D1
- D1 pad 1: row5 -> row0
- D10 pad 1: row2 -> row3
- D11 pad 1: row1 -> row4
- D12 pad 1: row0 -> row5
- D13 pad 1: row5 -> row0
- D14 pad 1: row4 -> row1
- D15 pad 1: row3 -> row2
- D16 pad 1: row2 -> row3
- D17 pad 1: row1 -> row4
- D18 pad 1: row0 -> row5
- D19 pad 1: row5 -> row0
- D2 pad 1: row4 -> row1
- D20 pad 1: row4 -> row1
- D21 pad 1: row3 -> row2
- D22 pad 1: row2 -> row3
- D23 pad 1: row1 -> row4
- D24 pad 1: row0 -> row5
- D25 pad 1: row5 -> row0
- D26 pad 1: row4 -> row1
- D27 pad 1: row3 -> row2
- D28 pad 1: row2 -> row3
- D29 pad 1: row1 -> row4
- D3 pad 1: row3 -> row2
- D30 pad 1: row0 -> row5
- D31 pad 1: row5 -> row0
- D32 pad 1: row4 -> row1
- D33 pad 1: row3 -> row2
- D34 pad 1: row2 -> row3
- D35 pad 1: row1 -> row4
- D36 pad 1: row0 -> row5
- D37 pad 1: row5 -> row0
- D38 pad 1: row4 -> row1
- D39 pad 1: row3 -> row2
- D4 pad 1: row2 -> row3
- D40 pad 1: row2 -> row3
- D41 pad 1: row1 -> row4
- D42 pad 1: row0 -> row5
- D5 pad 1: row1 -> row4
- D6 pad 1: row0 -> row5
- D7 pad 1: row5 -> row0
- D8 pad 1: row4 -> row1
- D9 pad 1: row3 -> row2
- LED1 pad 2: (no net) -> LED_36
- LED1 pad 4: (no net) -> LED_35
- LED10 pad 2: (no net) -> LED_33
- LED10 pad 4: (no net) -> LED_32
- LED11 pad 2: (no net) -> LED_19
- LED11 pad 4: (no net) -> LED_18
- LED12 pad 2: (no net) -> LED_5
- LED12 pad 4: (no net) -> LED_4
- LED13 pad 2: (no net) -> LED_32
- LED13 pad 4: (no net) -> LED_31
- LED14 pad 2: (no net) -> LED_18
- LED14 pad 4: (no net) -> LED_17
- LED15 pad 2: (no net) -> LED_4
- LED15 pad 4: (no net) -> LED_3
- LED16 pad 2: (no net) -> LED_31
- LED16 pad 4: (no net) -> LED_30
- LED17 pad 2: (no net) -> LED_17
- LED17 pad 4: (no net) -> LED_16
- LED18 pad 2: (no net) -> LED_3
- LED18 pad 4: (no net) -> LED_2
- LED19 pad 2: (no net) -> LED_30
- LED19 pad 4: (no net) -> LED_29
- LED2 pad 2: (no net) -> LED_22
- LED2 pad 4: (no net) -> LED_21
- LED20 pad 2: (no net) -> LED_16
- LED20 pad 4: (no net) -> LED_15
- LED21 pad 2: (no net) -> LED_2
- LED21 pad 4: (no net) -> LED_1
- LED22 pad 2: (no net) -> LED_37
- LED22 pad 4: (no net) -> LED_36
- LED23 pad 2: (no net) -> LED_23
- LED23 pad 4: (no net) -> LED_22
- LED24 pad 2: (no net) -> LED_9
- LED24 pad 4: (no net) -> LED_8
- LED25 pad 2: (no net) -> LED_38
- LED25 pad 4: (no net) -> LED_37
- LED26 pad 2: (no net) -> LED_24
- LED26 pad 4: (no net) -> LED_23
- LED27 pad 2: (no net) -> LED_10
- LED27 pad 4: (no net) -> LED_9
- LED28 pad 2: (no net) -> LED_39
- LED28 pad 4: (no net) -> LED_38
- LED29 pad 2: (no net) -> LED_25
- LED29 pad 4: (no net) -> LED_24
- LED3 pad 2: (no net) -> LED_8
- LED3 pad 4: (no net) -> LED_7
- LED30 pad 2: (no net) -> LED_11
- LED30 pad 4: (no net) -> LED_10
- LED31 pad 2: (no net) -> LED_40
- LED31 pad 4: (no net) -> LED_39
- LED32 pad 2: (no net) -> LED_26
- LED32 pad 4: (no net) -> LED_25
- LED33 pad 2: (no net) -> LED_12
- LED33 pad 4: (no net) -> LED_11
- LED34 pad 2: (no net) -> LED_41
- LED34 pad 4: (no net) -> LED_40
- LED35 pad 2: (no net) -> LED_27
- LED35 pad 4: (no net) -> LED_26
- LED36 pad 2: (no net) -> LED_13
- LED36 pad 4: (no net) -> LED_12
- LED37 pad 2: (no net) -> LED_42
- LED37 pad 4: (no net) -> LED_41
- LED38 pad 2: (no net) -> LED_28
- LED38 pad 4: (no net) -> LED_27
- LED39 pad 2: (no net) -> LED_14
- LED39 pad 4: (no net) -> LED_13
- LED4 pad 2: (no net) -> LED_35
- LED4 pad 4: (no net) -> LED_34
- LED40 pad 4: (no net) -> LED_42
- LED41 pad 2: (no net) -> LED_29
- LED41 pad 4: (no net) -> LED_28
- LED42 pad 2: (no net) -> LED_13
- LED42 pad 4: (no net) -> LED_14
- LED5 pad 2: (no net) -> LED_21
- LED5 pad 4: (no net) -> LED_20
- LED6 pad 2: (no net) -> LED_7
- LED6 pad 4: (no net) -> LED_6
- LED7 pad 2: (no net) -> LED_34
- LED7 pad 4: (no net) -> LED_33
- LED8 pad 2: (no net) -> LED_20
- LED8 pad 4: (no net) -> LED_19
- LED9 pad 2: (no net) -> LED_6
- LED9 pad 4: (no net) -> LED_5
- MCU1 pad 10: row3 -> row4
- MCU1 pad 11: row4 -> row5
- MCU1 pad 13: encC -> col0
- MCU1 pad 14: encA -> col1
- MCU1 pad 15: B3 -> col2
- MCU1 pad 16: B1 -> col3
- MCU1 pad 17: col3 -> col4
- MCU1 pad 18: col2 -> col5
- MCU1 pad 19: col1 -> col6
- MCU1 pad 20: col0 -> LED_1
- MCU1 pad 6: scl -> row0
- MCU1 pad 7: row0 -> row1
- MCU1 pad 8: row1 -> row2
- MCU1 pad 9: row2 -> row3
Routing:
- added copper zone on B.Cu, net GND
- added copper zone on F.Cu, net GND
Other:
- board size 161.3 x 139.9 mm -> 163.4 x 159.9 mm
- board text added: "2025.11.06"
- board text added: "JLCJLCJLCJLC"
- board text added: "LED_1"
- board text added: "LED_10"
- board text added: "LED_11"
- board text added: "LED_12"
- board text added: "LED_13"
- board text added: "LED_14"
- board text added: "LED_15"
- board text added: "LED_16"
- board text added: "LED_17"
- board text added: "LED_18"
- board text added: "LED_19"
- board text added: "LED_2"
- board text added: "LED_20"
- board text added: "LED_21"
- board text added: "LED_22"
- board text added: "LED_23"
- board text added: "LED_24"
- board text added: "LED_25"
- board text added: "LED_26"
- board text added: "LED_27"
- board text added: "LED_28"
- board text added: "LED_29"
- board text added: "LED_3"
- board text added: "LED_30"
- board text added: "LED_31"
- board text added: "LED_32"
- board text added: "LED_33"
- board text added: "LED_34"
- board text added: "LED_35"
- board text added: "LED_36"
- board text added: "LED_37"
- board text added: "LED_38"
- board text added: "LED_39"
- board text added: "LED_4"
- board text added: "LED_40"
- board text added: "LED_41"
- board text added: "LED_42"
- board text added: "LED_5"
- board text added: "LED_6"
- board text added: "LED_7"
- board text added: "LED_8"
- board text added: "LED_9"
- board text added: "https://github.com/dieseltravis/travis-ergogen-2026"
- board text added: "made with ♥ in #ROC"
- board text added: "travis-ergogen-2026"

Commit message: updates
Parts:
- removed C40, C41, C42, C43: C_1206_3216Metric, C_1206_3216Metric
- removed D41, D42: D_1206_3216Metric, D_1206_3216Metric
- removed LED39, LED40, LED41, LED42: SK6812mini-e, travis:led_SK6812mini-e (per-key, single-side)
- removed S41, S42: Kailh MX Switch Sockets, travis:MX
- moved S24 108.1 mm to (130.1, 195.9), turned to 179 degrees
- moved D24 108.0 mm to (121.5, 201.9), turned to 89 degrees
- moved S18 106.2 mm to (110.0, 194.9), turned to 180 degrees
- moved S12 106.2 mm to (90.0, 196.3), turned to 181 degrees
- moved D12 106.0 mm to (81.7, 202.5), turned to 91 degrees
- moved D18 106.0 mm to (101.6, 201.0), turned to 90 degrees
- moved S36 87.9 mm to (171.5, 178.1), turned to 177 degrees
- moved D36 87.7 mm to (162.8, 183.8), turned to 87 degrees
- moved S30 87.6 mm to (150.8, 176.2), turned to 178 degrees
- moved D30 87.4 mm to (142.2, 182.0), turned to 88 degrees
- moved S35 85.6 mm to (160.1, 198.4), turned to 176 degrees
- moved D35 85.3 mm to (151.2, 203.9), turned to 86 degrees
- moved LED28 84.2 mm to (88.4, 107.1)
- moved LED34 84.2 mm to (131.6, 106.8)
- moved LED31 84.2 mm to (110.0, 105.7)
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Connections:
- D10 pad 1: row3 -> row4
- D10 pad 2: matrix_col1_row3 -> matrix_col1_row4
- D11 pad 1: row4 -> row5
- D11 pad 2: matrix_col1_row4 -> matrix_col1_row5
- D12 pad 1: row5 -> row0
- D12 pad 2: matrix_col1_row5 -> matrix_col2_row0
- D13 pad 1: row0 -> row1
- D13 pad 2: matrix_col2_row0 -> matrix_col2_row1
- D14 pad 1: row1 -> row2
- D14 pad 2: matrix_col2_row1 -> matrix_col2_row2
- D15 pad 1: row2 -> row3
- D15 pad 2: matrix_col2_row2 -> matrix_col2_row3
- D16 pad 1: row3 -> row4
- D16 pad 2: matrix_col2_row3 -> matrix_col2_row4
- D17 pad 1: row4 -> row5
- D17 pad 2: matrix_col2_row4 -> matrix_col2_row5
- D18 pad 1: row5 -> row0
- D18 pad 2: matrix_col2_row5 -> matrix_col3_row0
- D19 pad 1: row0 -> row1
- D19 pad 2: matrix_col3_row0 -> matrix_col3_row1
- D20 pad 1: row1 -> row2
- D20 pad 2: matrix_col3_row1 -> matrix_col3_row2
- D21 pad 1: row2 -> row3
- D21 pad 2: matrix_col3_row2 -> matrix_col3_row3
- D22 pad 1: row3 -> row4
- D22 pad 2: matrix_col3_row3 -> matrix_col3_row4
- D23 pad 1: row4 -> row5
- D23 pad 2: matrix_col3_row4 -> matrix_col3_row5
- D24 pad 1: row5 -> row0
- D24 pad 2: matrix_col3_row5 -> matrix_col4_row0
- D25 pad 1: row0 -> row1
- D25 pad 2: matrix_col4_row0 -> matrix_col4_row1
- D26 pad 1: row1 -> row2
- D26 pad 2: matrix_col4_row1 -> matrix_col4_row2
- D27 pad 1: row2 -> row3
- D27 pad 2: matrix_col4_row2 -> matrix_col4_row3
- D28 pad 1: row3 -> row4
- D28 pad 2: matrix_col4_row3 -> matrix_col4_row4
- D29 pad 1: row4 -> row5
- D29 pad 2: matrix_col4_row4 -> matrix_col4_row5
- D30 pad 1: row5 -> row1
- D30 pad 2: matrix_col4_row5 -> matrix_col5_row1
- D31 pad 1: row0 -> row2
- D31 pad 2: matrix_col5_row0 -> matrix_col5_row2
- D32 pad 1: row1 -> row3
- D32 pad 2: matrix_col5_row1 -> matrix_col5_row3
- D33 pad 1: row2 -> row4
- D33 pad 2: matrix_col5_row2 -> matrix_col5_row4
- D34 pad 1: row3 -> row5
- D34 pad 2: matrix_col5_row3 -> matrix_col5_row5
- D35 pad 1: row4 -> row0
- D35 pad 2: matrix_col5_row4 -> matrix_col6_row0
- D36 pad 1: row5 -> row1
- D36 pad 2: matrix_col5_row5 -> matrix_col6_row1
- D37 pad 1: row0 -> row2
- D37 pad 2: matrix_col6_row0 -> matrix_col6_row2
- D38 pad 1: row1 -> row3
- D38 pad 2: matrix_col6_row1 -> matrix_col6_row3
- D39 pad 1: row2 -> row4
- D39 pad 2: matrix_col6_row2 -> matrix_col6_row4
- D40 pad 1: row3 -> row5
- D40 pad 2: matrix_col6_row3 -> matrix_col6_row5
- D7 pad 1: row0 -> row1
- D7 pad 2: matrix_col1_row0 -> matrix_col1_row1
- D8 pad 1: row1 -> row2
- D8 pad 2: matrix_col1_row1 -> matrix_col1_row2
- D9 pad 1: row2 -> row3
- D9 pad 2: matrix_col1_row2 -> matrix_col1_row3
- LED22 pad 2: LED_37 -> LED_23
- LED22 pad 4: LED_36 -> LED_22
- LED23 pad 2: LED_23 -> LED_9
- LED23 pad 4: LED_22 -> LED_8
- LED24 pad 2: LED_9 -> LED_24
- LED24 pad 4: LED_8 -> LED_23
- LED25 pad 2: LED_38 -> LED_10
- LED25 pad 4: LED_37 -> LED_9
- LED26 pad 2: LED_24 -> LED_39
- LED26 pad 4: LED_23 -> LED_38
- LED27 pad 2: LED_10 -> LED_25
- LED27 pad 4: LED_9 -> LED_24
- LED28 pad 2: LED_39 -> LED_11
- LED28 pad 4: LED_38 -> LED_10
- LED29 pad 2: LED_25 -> LED_40
- LED29 pad 4: LED_24 -> LED_39
- LED30 pad 2: LED_11 -> LED_26
- LED30 pad 4: LED_10 -> LED_25
- LED31 pad 2: LED_40 -> LED_12
- LED31 pad 4: LED_39 -> LED_11
- LED32 pad 2: LED_26 -> LED_41
- LED32 pad 4: LED_25 -> LED_40
- LED33 pad 2: LED_12 -> LED_27
- LED33 pad 4: LED_11 -> LED_26
- LED34 pad 2: LED_41 -> LED_13
- LED34 pad 4: LED_40 -> LED_12
- LED35 pad 2: LED_27 -> LED_28
- LED35 pad 4: LED_26 -> LED_27
- LED36 pad 2: LED_13 -> LED_14
- LED36 pad 4: LED_12 -> LED_13
- LED37 pad 2: LED_42 -> LED_29
- LED37 pad 4: LED_41 -> LED_28
- LED38 pad 2: LED_28 -> LED_13
- LED38 pad 4: LED_27 -> LED_14
- S10 pad 2: matrix_col1_row3 -> matrix_col1_row4
- S11 pad 2: matrix_col1_row4 -> matrix_col1_row5
- S12 pad 1: col1 -> col2
- S12 pad 2: matrix_col1_row5 -> matrix_col2_row0
- S13 pad 2: matrix_col2_row0 -> matrix_col2_row1
- S14 pad 2: matrix_col2_row1 -> matrix_col2_row2
- S15 pad 2: matrix_col2_row2 -> matrix_col2_row3
- S16 pad 2: matrix_col2_row3 -> matrix_col2_row4
- S17 pad 2: matrix_col2_row4 -> matrix_col2_row5
- S18 pad 1: col2 -> col3
- S18 pad 2: matrix_col2_row5 -> matrix_col3_row0
- S19 pad 2: matrix_col3_row0 -> matrix_col3_row1
- S20 pad 2: matrix_col3_row1 -> matrix_col3_row2
- S21 pad 2: matrix_col3_row2 -> matrix_col3_row3
- S22 pad 2: matrix_col3_row3 -> matrix_col3_row4
- S23 pad 2: matrix_col3_row4 -> matrix_col3_row5
- S24 pad 1: col3 -> col4
- S24 pad 2: matrix_col3_row5 -> matrix_col4_row0
- S25 pad 2: matrix_col4_row0 -> matrix_col4_row1
- S26 pad 2: matrix_col4_row1 -> matrix_col4_row2
- S27 pad 2: matrix_col4_row2 -> matrix_col4_row3
- S28 pad 2: matrix_col4_row3 -> matrix_col4_row4
- S29 pad 2: matrix_col4_row4 -> matrix_col4_row5
- S30 pad 1: col4 -> col5
- S30 pad 2: matrix_col4_row5 -> matrix_col5_row1
- S31 pad 2: matrix_col5_row0 -> matrix_col5_row2
- S32 pad 2: matrix_col5_row1 -> matrix_col5_row3
- S33 pad 2: matrix_col5_row2 -> matrix_col5_row4
- S34 pad 2: matrix_col5_row3 -> matrix_col5_row5
- S35 pad 1: col5 -> col6
- S35 pad 2: matrix_col5_row4 -> matrix_col6_row0
- S36 pad 1: col5 -> col6
- S36 pad 2: matrix_col5_row5 -> matrix_col6_row1
- S37 pad 2: matrix_col6_row0 -> matrix_col6_row2
- S38 pad 2: matrix_col6_row1 -> matrix_col6_row3
- S39 pad 2: matrix_col6_row2 -> matrix_col6_row4
- S40 pad 2: matrix_col6_row3 -> matrix_col6_row5
- S7 pad 2: matrix_col1_row0 -> matrix_col1_row1
- S8 pad 2: matrix_col1_row1 -> matrix_col1_row2
- S9 pad 2: matrix_col1_row2 -> matrix_col1_row3
Other:
- board size 163.4 x 159.9 mm -> 163.7 x 159.6 mm
- board text added: "2026.01.14"
- board text removed: "2025.11.06"
- board text removed: "LED_36"
- board text removed: "LED_37"
- board text removed: "LED_41"
- board text removed: "LED_42"
- board text removed: "S41"
- board text removed: "S42"
