File: output/pcbs/travis_erg2026.kicad_pcb (KiCad board)
At the start: 2 copper layers, 167.2 x 170.9 mm, 184 parts

Commit message: plate
Connections:
- MCU1 pad 13: row5 -> row0
- MCU1 pad 14: row4 -> row1
- MCU1 pad 15: row3 -> row2
- MCU1 pad 16: row2 -> row3
- MCU1 pad 17: row1 -> row4
- MCU1 pad 18: row0 -> row5

Commit message: trrs, corners
Parts:
- added TRRS1: , ceoloide:trrs_pj320a, F.Cu at (148.9, 57.3)
- moved HOLE4 9.90 mm to (181.8, 214.8)
- moved HOLE6 9.90 mm to (38.3, 215.8)
Connections:
- MCU1 pad 19: B6 -> col0
- MCU1 pad 2: D3 -> TX
- MCU1 pad 20: col0 -> col1
- MCU1 pad 21: col1 -> col2
- MCU1 pad 22: col2 -> col3
- MCU1 pad 23: col3 -> col4
- MCU1 pad 24: col4 -> col6
- MCU1 pad 25: col5 -> col7
- MCU1 pad 26: col6 -> F4
- MCU1 pad 3: D2 -> RX
Other:
- board size 167.2 x 170.9 mm -> 167.2 x 169.8 mm

Commit message: trrs data sheet
Parts:
- added TRRS2: , ceoloide:trrs_pj320a, F.Cu at (152.0, 57.4)
- moved TRRS1 3.36 mm to (145.6, 57.0)
Changed lines of the file:
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@@
   (title_block
     (title "travis_erg2026")
-    (date "2026-02-08")
+    (date "2026-02-10")
     (rev "2026.02.02")
     (company "Travis Hardiman")
@@
   (footprint "ceoloide:trrs_pj320a"
     (layer "F.Cu")
-    (at 148.94055290000003 57.30281700000004 -3.6)
+    (at 145.59957350000002 56.98602550000004 -3.6)
     (property "Reference" "TRRS1"
       (at 0 14.2 -3.6)
@@
     (pad 5 thru_hole oval (at -2.3 11.3 -3.6) (size 1.6 2.2) (drill oval 0.9 1.5) (layers "*.Cu" "*.Mask") (net 2 "TX"))
   )
+  (footprint "ceoloide:trrs_pj320a"
+    (layer "F.Cu")
+    (at 152.03866440000004 57.41100540000004 -3.6)
+    (property "Reference" "TRRS2"
+      (at 0 14.2 -3.6)
+      (layer "F.SilkS")
+      hide
+      (effects (font (size 1 1) (thickness 0.15)))
+    )
+    (fp_line (start 2.8 -2) (end -2.8 -2) (layer "Dwgs.User") (stroke (width 0.15) (type solid)))
+    (fp_line (start -2.8 0) (end -2.8 -2) (layer "Dwgs.User") (stroke (width 0.15) (type solid)))
+    (fp_line (start 2.8 0) (end 2.8 -2) (layer "Dwgs.User") (stroke (width 0.15) (type solid)))
+    (fp_line (start -3.05 0) (end -3.05 12.1) (layer "Dwgs.User") (stroke (width 0.15) (type solid)))
+    (fp_line (start 3.05 0) (end 3.05 12.1) (layer "Dwgs.User") (stroke (width 0.15) (type solid)))
+    (fp_line (start 3.05 12.1) (end -3.05 12.1) (layer "Dwgs.User") (stroke (width 0.15) (type solid)))
+    (fp_line (start 3.05 0) (end -3.05 0) (layer "Dwgs.User") (stroke (width 0.15) (type solid)))
+    (pad "" np_thru_hole circle (at 0 8.6 -3.6) (size 1.5 1.5) (drill 1.5) (layers "*.Cu" "*.Mask"))
+    (pad "" np_thru_hole circle (at 0 1.6 -3.6) (size 1.5 1.5) (drill 1.5) (layers "*.Cu" "*.Mask"))
+    (pad 2 thru_hole oval (at 2.3 3.2 -3.6) (size 1.6 2.2) (drill oval 0.9 1.5) (layers "*.Cu" "*.Mask") (net 4 "GND"))
+    (pad 3 thru_hole oval (at 2.3 6.2 -3.6) (size 1.6 2.2) (drill oval 0.9 1.5) (layers "*.Cu" "*.Mask") (net 2 "TX"))
+    (pad 4 thru_hole oval (at 2.3 10.2 -3.6) (size 1.6 2.2) (drill oval 0.9 1.5) (layers "*.Cu" "*.Mask") (net 26 "VCC"))
+    (pad 5 thru_hole oval (at -2.3 11.3 -3.6) (size 1.6 2.2) (drill oval 0.9 1.5) (layers "*.Cu" "*.Mask") (net 3 "RX"))
+  )
 (footprint "I2C_Breakout" (version 20210126) (generator pcbnew) (layer "F.Cu")
