File: output/pcbs/travis_erg2026-v3-round.kicad_pcb (KiCad board)
At the start: 2 copper layers, 167.2 x 170.9 mm, 184 parts

Commit message: trrs, corners
Routing:
- net GND: track 142.3 -> 143.4 mm, vias 49 -> 57
